Commit message: added meshes, urdf, config to the repo

File: urdf/arm (copy).urdf (robot description, URDF)
Before this commit: robot arm, 17 links, 16 joints
Links:
- link base_link: geometry collision box size=90.5 90.2 80.1; visual mesh filename=package://armando_description/meshes/base_link.stl scale=0.001 0.001 0.001
- link base_turn: geometry collision box size=60.1 78.3 7.1; visual mesh filename=package://armando_description/meshes/base_turn.stl scale=0.001 0.001 0.001
- link base_turn_rot: geometry collision box size=56.1 55.7 20.8; visual mesh filename=package://armando_description/meshes/base_turn_table_rot.stl scale=0.001 0.001 0.001
- link crawer_base: geometry collision box size=104.1 57.9 5.1; visual mesh filename=package://armando_description/meshes/the_crawer_base.stl scale=0.001 0.001 0.001
- link crawer_left: geometry collision box size=63 31.3 40.9; visual mesh filename=package://armando_description/meshes/the_crawer.stl scale=0.001 0.001 0.001
- link crawer_right: geometry collision box size=63 31.3 40.9; visual mesh filename=package://armando_description/meshes/the_crawer.stl scale=0.001 0.001 0.001
- link dyn2: geometry collision box size=5.1 3.3 4.1; visual mesh filename=package://armando_description/meshes/dyn.stl scale=0.01 0.01 0.01
- link dyn3: geometry collision box size=5.1 3.3 4.1; visual mesh filename=package://armando_description/meshes/dyn.stl scale=0.01 0.01 0.01
- link dyn4: geometry collision box size=5.1 3.3 4.1; visual mesh filename=package://armando_description/meshes/dyn.stl scale=0.01 0.01 0.01
- link dyn5: geometry collision box size=5.1 3.3 4.1; visual mesh filename=package://armando_description/meshes/dyn.stl scale=0.01 0.01 0.01
- link f4: geometry collision box size=48.1 91.7 28.7; visual mesh filename=package://armando_description/meshes/f4_n_f3.stl scale=0.001 0.001 0.001
- link f5: geometry collision box size=48.1 91.7 28.7; visual mesh filename=package://armando_description/meshes/f4_n_f3.stl scale=0.001 0.001 0.001
- link wrist: geometry collision box size=48.3 54.8 43.1; visual mesh filename=package://armando_description/meshes/wrist.stl scale=0.001 0.001 0.001
