Commit message: upload all current files

File: urdf/arm_old.urdf.xacro (robot description, xacro)
@@ -1,4 +1,4 @@
 <?xml version="1.0"?>
-<robot name="arm">
+<robot name="arm" xmlns:xacro="http://www.ros.org/wiki/xacro">
   <material name="red">
     <color rgba="1 0 0 1"/>
@@ -7,12 +7,12 @@
     <visual>
       <geometry>
-        <mesh filename="package://armando_description/meshes/base_link.stl" scale="0.001 0.001 0.001"/>
-      </geometry>
-      <origin rpy="0 0 0" xyz="0 0 0"/>
-      <material name="red"/>
-    </visual>
-    <collision>
-      <geometry>
-        <box size="90.5 90.2 80.1" />
+        <mesh filename="model://armando_description/meshes/base_link.stl" scale="0.001 0.001 0.001"/>
+      </geometry>
+      <origin rpy="0 0 0" xyz="0 0 0"/>
+      <material name="red"/>
+    </visual>
+    <collision>
+      <geometry>
+        <mesh filename="model://armando_description/meshes/base_link.stl" scale="0.001 0.001 0.001"/>
       </geometry>
       <origin rpy="0 0 0" xyz="0 0 0"/>
@@ -31,12 +31,12 @@
     <visual>
       <geometry>
-        <mesh filename="package://armando_description/meshes/base_turn.stl" scale="0.001 0.001 0.001"/>
-      </geometry>
-      <origin rpy="0 0 0" xyz="0 0 0"/>
-      <material name="red"/>
-    </visual>
-    <collision>
-      <geometry>
-          <box size="60.1 78.3 7.1" />
+        <mesh filename="model://armando_description/meshes/base_turn.stl" scale="0.001 0.001 0.001"/>
+      </geometry>
+      <origin rpy="0 0 0" xyz="0 0 0"/>
+      <material name="red"/>
+    </visual>
+    <collision>
+      <geometry>
+          <mesh filename="model://armando_description/meshes/base_turn.stl" scale="0.001 0.001 0.001"/>
         </geometry>
       <origin rpy="0 0 0" xyz="0 0 0"/>
@@ -57,11 +57,11 @@
     <visual>
       <geometry>
-        <mesh filename="package://armando_description/meshes/base_turn_table_rot.stl" scale="0.001 0.001 0.001"/>
-      </geometry>
-      <material name="red"/>
-    </visual>
-    <collision>
-      <geometry>
-          <box size="56.1 55.7 20.8" />
+        <mesh filename="model://armando_description/meshes/base_turn_table_rot.stl" scale="0.001 0.001 0.001"/>
+      </geometry>
+      <material name="red"/>
+    </visual>
+    <collision>
+      <geometry>
+          <mesh filename="model://armando_description/meshes/base_turn_table_rot.stl" scale="0.001 0.001 0.001"/>
         </geometry>
       <origin rpy="0 0 0" xyz="0 0 0"/>
@@ -80,11 +80,11 @@
     <visual>
       <geometry>
-        <mesh filename="package://armando_description/meshes/dyn.stl" scale="0.01 0.01 0.01"/>
-      </geometry>
-      <origin rpy="0 0 0" xyz="0 0 0"/>
-    </visual>
-    <collision>
-      <geometry>
-          <box size="5.1 3.3 4.1" />
+        <mesh filename="model://armando_description/meshes/dyn.stl" scale="0.01 0.01 0.01"/>
+      </geometry>
+      <origin rpy="0 0 0" xyz="0 0 0"/>
+    </visual>
+    <collision>
+      <geometry>
+          <mesh filename="model://armando_description/meshes/dyn.stl" scale="0.01 0.01 0.01"/>
         </geometry>
       <origin rpy="0 0 0" xyz="0 0 0"/>
@@ -112,12 +112,12 @@
     <visual>
       <geometry>
-        <mesh filename="package://armando_description/meshes/f4_n_f3.stl" scale="0.001 0.001 0.001"/>
-      </geometry>
-      <origin rpy="0 0 0" xyz="0 0 0"/>
-      <material name="red"/>
-    </visual>
-    <collision>
-      <geometry>
-          <box size="48.1 91.7 28.7" />
+        <mesh filename="model://armando_description/meshes/f4_n_f3.stl" scale="0.001 0.001 0.001"/>
+      </geometry>
+      <origin rpy="0 0 0" xyz="0 0 0"/>
+      <material name="red"/>
+    </visual>
+    <collision>
+      <geometry>
+          <mesh filename="model://armando_description/meshes/f4_n_f3.stl" scale="0.001 0.001 0.001"/>
         </geometry>
       <origin rpy="0 0 0" xyz="0 0 0"/>
@@ -136,11 +136,11 @@
     <visual>
       <geometry>
-        <mesh filename="package://armando_description/meshes/dyn.stl" scale="0.01 0.01 0.01"/>
-      </geometry>
-      <origin rpy="0 0 0" xyz="0 0 0"/>
-    </visual>
-    <collision>
-      <geometry>
-          <box size="5.1 3.3 4.1" />
+        <mesh filename="model://armando_description/meshes/dyn.stl" scale="0.01 0.01 0.01"/>
+      </geometry>
+      <origin rpy="0 0 0" xyz="0 0 0"/>
+    </visual>
+    <collision>
+      <geometry>
+          <mesh filename="model://armando_description/meshes/dyn.stl" scale="0.01 0.01 0.01"/>
         </geometry>
       <origin rpy="0 0 0" xyz="0 0 0"/>
@@ -168,12 +168,12 @@
     <visual>
       <geometry>
-        <mesh filename="package://armando_description/meshes/f4_n_f3.stl" scale="0.001 0.001 0.001"/>
-      </geometry>
-      <origin rpy="0 0 0" xyz="0 0 0"/>
-      <material name="red"/>
-    </visual>
-    <collision>
-      <geometry>
-          <box size="48.1 91.7 28.7" />
+        <mesh filename="model://armando_description/meshes/f4_n_f3.stl" scale="0.001 0.001 0.001"/>
+      </geometry>
+      <origin rpy="0 0 0" xyz="0 0 0"/>
+      <material name="red"/>
+    </visual>
+    <collision>
+      <geometry>
+          <mesh filename="model://armando_description/meshes/f4_n_f3.stl" scale="0.001 0.001 0.001"/>
         </geometry>
       <origin rpy="0 0 0" xyz="0 0 0"/>
@@ -191,11 +191,11 @@
     <visual>
       <geometry>
-        <mesh filename="package://armando_description/meshes/dyn.stl" scale="0.01 0.01 0.01"/>
-      </geometry>
-      <origin rpy="0 0 0" xyz="0 0 0"/>
-    </visual>
-    <collision>
-      <geometry>
-          <box size="5.1 3.3 4.1" />
+        <mesh filename="model://armando_description/meshes/dyn.stl" scale="0.01 0.01 0.01"/>
+      </geometry>
+      <origin rpy="0 0 0" xyz="0 0 0"/>
+    </visual>
+    <collision>
+      <geometry>
+          <mesh filename="model://armando_description/meshes/dyn.stl" scale="0.01 0.01 0.01"/>
         </geometry>
       <origin rpy="0 0 0" xyz="0 0 0"/>
@@ -223,12 +223,12 @@
     <visual>
       <geometry>
-        <mesh filename="package://armando_description/meshes/wrist.stl" scale="0.001 0.001 0.001"/>
-      </geometry>
-      <origin rpy="0 0 0" xyz="0 0 0"/>
-      <material name="red"/>
-    </visual>
-    <collision>
-      <geometry>
-        <box size="48.3 54.8 43.1" />
+        <mesh filename="model://armando_description/meshes/wrist.stl" scale="0.001 0.001 0.001"/>
+      </geometry>
+      <origin rpy="0 0 0" xyz="0 0 0"/>
+      <material name="red"/>
+    </visual>
+    <collision>
+      <geometry>
+        <mesh filename="model://armando_description/meshes/wrist.stl" scale="0.001 0.001 0.001"/>
       </geometry>
       <origin rpy="0 0 0" xyz="0 0 0"/>
@@ -247,11 +247,11 @@
     <visual>
       <geometry>
-        <mesh filename="package://armando_description/meshes/dyn.stl" scale="0.01 0.01 0.01"/>
-      </geometry>
-      <origin rpy="0 0 0" xyz="0 0 0"/>
-    </visual>
-    <collision>
-      <geometry>
-          <box size="5.1 3.3 4.1" />
+        <mesh filename="model://armando_description/meshes/dyn.stl" scale="0.01 0.01 0.01"/>
+      </geometry>
+      <origin rpy="0 0 0" xyz="0 0 0"/>
+    </visual>
+    <collision>
+      <geometry>
+          <mesh filename="model://armando_description/meshes/dyn.stl" scale="0.01 0.01 0.01"/>
         </geometry>
       <origin rpy="0 0 0" xyz="0 0 0"/>
@@ -279,12 +279,12 @@
     <visual>
       <geometry>
-        <mesh filename="package://armando_description/meshes/the_crawer_base.stl" scale="0.001 0.001 0.001"/>
-      </geometry>
-      <origin rpy="0 0 0" xyz="0 0 0"/>
-      <material name="red"/>
-    </visual>
-    <collision>
-      <geometry>
-          <box size="104.1 57.9 5.1" />
+        <mesh filename="model://armando_description/meshes/the_crawer_base.stl" scale="0.001 0.001 0.001"/>
+      </geometry>
+      <origin rpy="0 0 0" xyz="0 0 0"/>
+      <material name="red"/>
+    </visual>
+    <collision>
+      <geometry>
+          <mesh filename="model://armando_description/meshes/the_crawer_base.stl" scale="0.001 0.001 0.001"/>
         </geometry>
       <origin rpy="0 0 0" xyz="0 0 0"/>
@@ -303,5 +303,5 @@
     <visual>
       <geometry>
-        <mesh filename="package://armando_description/meshes/the_crawer.stl" scale="0.001 0.001 0.001"/>
+        <mesh filename="model://armando_description/meshes/the_crawer.stl" scale="0.001 0.001 0.001"/>
       </geometry>
       <origin rpy="0 0 0" xyz="0 0 0"/>
@@ -312,5 +312,5 @@
     <collision>
       <geometry>
-          <box size="63 31.3 40.9" />
+          <mesh filename="model://armando_description/meshes/the_crawer.stl" scale="0.001 0.001 0.001"/>
         </geometry>
       <origin rpy="0 0 0" xyz="0 0 0"/>
@@ -329,5 +329,5 @@
     <visual>
       <geometry>
-        <mesh filename="package://armando_description/meshes/the_crawer.stl" scale="0.001 0.001 0.001"/>
+        <mesh filename="model://armando_description/meshes/the_crawer.stl" scale="0.001 0.001 0.001"/>
       </geometry>
       <origin rpy="0 0 0" xyz="0 0 0"/>
@@ -338,12 +338,19 @@
     <collision>
       <geometry>
-          <box size="63 31.3 40.9" />
-        </geometry>
-      <origin rpy="0 0 0" xyz="0 0 0"/>
-    </collision>
-    <inertial>
-      <mass value="0.1"/>
-      <inertia ixx="6.90013881e-05" ixy="0.0" ixz="0.0" iyy="1.24554875e-04" iyz="0.0" izz="1.04295793e-04"/>
-    </inertial>
-  </link>
+          <mesh filename="model://armando_description/meshes/the_crawer.stl" scale="0.001 0.001 0.001"/>
+        </geometry>
+      <origin rpy="0 0 0" xyz="0 0 0"/>
+    </collision>
+    <inertial>
+      <mass value="0.1"/>
+      <inertia ixx="6.90013881e-05" ixy="0.0" ixz="0.0" iyy="1.24554875e-04" iyz="0.0" izz="1.04295793e-04"/>
+    </inertial>
+  </link>
+  <xacro:include filename="$(find armando_description)/urdf/armando_hardware_interface.xacro"/>
+  <xacro:armando_hardware_interface/>
+  <gazebo>
+    <plugin filename="gz_ros2_control-system" name="gz_ros2_control::GazeboSimROS2ControlPlugin">
+     <parameters>$(find armando_description)/config/arm_position_controllers.yaml</parameters>
+    </plugin>
+  </gazebo>
 </robot>

Commit message: Update arm_old.urdf.xacro

File: urdf/arm_old.urdf.xacro (robot description, xacro)
@@ -22,4 +22,17 @@
       <inertia ixx="1.06682889e+08" ixy="0.0" ixz="0.0" iyy="9.92165844e+07" iyz="0.0" izz="1.26939175e+08"/>
     </inertial>
+  </link>
+  <joint name="camera_joint" type="fixed">
+      <parent link="base_link"/>
+      <child link="camera_link"/>
+      <origin xyz="0 0 0.020" rpy="0.0 -1.57 0.0"/>
+  </joint>
+  <link name="camera_link">
+      <visual>
+          <geometry>
+              <box size="0.025 0.055 0.025"/>
+          </geometry>
+          <material name="blu"/>
+      </visual>
   </link>
   <joint name="base_1_2" type="fixed">

Commit message: Update arm_old.urdf.xacro

File: urdf/arm_old.urdf.xacro (robot description, xacro)
@@ -3,4 +3,7 @@
   <material name="red">
     <color rgba="1 0 0 1"/>
+  </material>
+  <material name="blu">
+    <color rgba="0 0 1 1"/>
   </material>
   <link name="base_link">
